Commit message: urdf accurate now

File: urdf/5DOF.urdf (robot description, URDF)
Before this commit: robot 5DOF, 9 links, 8 joints
Links:
- link Link1: mass 0.0289860326782574 -> None; geometry visual mesh filename=package://5DOF/meshes/Link1.STL
- link Link2: mass 0.0727270945890701 -> None; geometry visual mesh filename=package://5DOF/meshes/Link2.STL
- link Link3: mass 0.090914548707032 -> None; geometry visual mesh filename=package://5DOF/meshes/Link3.STL
- link Link4: mass 0.0257561871549524 -> None; geometry visual mesh filename=package://5DOF/meshes/Link4.STL
- link Link5: mass 0.00713826707604841 -> None; geometry visual mesh filename=package://5DOF/meshes/Link5.STL
Joints:
- removed joint world_to_base_link
- added joint world_to_thor1: type fixed, parent world, child base_link, origin xyz=-0.052 -0.2125 0 rpy=0 0 3.1415, axis 0 0 1
- joint Thor/1: origin xyz=0.1036 -0.05084 0.03635 rpy=1.5708 0 -0.025571 -> xyz=-0.052 -0.2125 0 rpy=1.5708 0 0; parent base_link -> world
- joint Thor/2: axis 0 0 -1 -> 0 0 1; origin xyz=-0.0019997 -0.031718 0.072325 rpy=0 0 -2.8294 -> xyz=-0.0019997 -0.031718 0.072325 rpy=0 0 0
- joint Thor/3: axis 0 1 0 -> 0 -1 0; origin xyz=-0.2774 0 -0.015403 rpy=1.5708 0 1.2521 -> xyz=-0.2774 0 -0.015403 rpy=1.5708 0 0
- joint Thor/4: origin xyz=-0.30216 -0.052613 0.00078978 rpy=0 -0.3981 0 -> xyz=-0.30216 -0.052613 0.00078978 rpy=0 3.1415 0
- joint Thor/6: axis 0 0 -1 -> 0 0 1; origin xyz=0.00016534 0.050763 0.0019121 rpy=-1.5708 0.71678 -1.5708 -> xyz=0.00016534 0.050763 0.0019121 rpy=-1.5708 -1.5708 -1.5708

Commit message: added tip and base transform

File: urdf/5DOF.urdf (robot description, URDF)
Before this commit: robot 5DOF, 9 links, 8 joints
Links:
- link base_link: mass 0.127147471977805 -> None; geometry visual mesh filename=package://5DOF/meshes/base_link.STL
Joints:
- joint Link5_to_tip: origin xyz=0 0 0 rpy=0 0 0 -> xyz=0 0 .042 rpy=0 0 0
- joint Thor/1: origin xyz=-0.052 -0.2125 0 rpy=1.5708 0 0 -> xyz=-0.052 -0.2125 .0356 rpy=1.5708 0 0
- joint Thor/4: axis 0 1 0 -> 0 -1 0
